File: Hardware/KiCAD/USBMuxV1/USBMuxV1.kicad_pcb (KiCad board)
At the start: 4 copper layers, 27 parts, among them J1 USB_B_Micro, J10 USB_A, J2 USB_A, J3 USB_A, J4 USB_A, J5 USB_A, J6 DF51K-16DP-XXXX, J7 USB_A, J8 USB_A, J9 USB_A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

Commit message: Finish routing
Parts:
- removed H1, H2: MountingHole_Pad, MountingHole:MountingHole_3.2mm_M3_Pad_Via
Routing:
- net Bank1OE: track 0.00 -> 49.0 mm, vias 0 -> 2
- net Bank3OE: track 0.00 -> 45.5 mm, vias 0 -> 2
- net Bank1Switch: track 0.00 -> 44.1 mm
- net Bank3Switch: track 0.00 -> 40.5 mm, vias 0 -> 1
- net GlobalD-: track 23.0 -> 58.5 mm, vias 0 -> 3
- net GlobalD+: track 23.5 -> 58.6 mm, vias 0 -> 3
- net Bank4OE: track 0.00 -> 29.0 mm, vias 0 -> 2
- net Bank2OE: track 0.00 -> 26.0 mm, vias 0 -> 2
- net Bank2Switch: track 0.00 -> 19.9 mm, vias 0 -> 2
- net Bank4Switch: track 0.00 -> 19.3 mm, vias 0 -> 2

Commit message: Update the PCB for round 1 of production
Connections:
- J1 pad 6: GND -> (no net)
Other:
- board outline added: 39 x 50 mm
